Commit message: updated urdf

File: suturo_manipulation_pr2_movit/config/pr2.urdf (robot description, URDF)
Before this commit: robot pr2, 95 links, 94 joints
Links:
- added link l_force_torque_adapter_link
- added link l_force_torque_link; visual cylinder length=0.0356 radius=0.0225
- link base_bellow_link: mass 1.0 -> 1
- link base_footprint: mass 1.0 -> 1
- link base_link: mass 116.0 -> 116
- link torso_lift_motor_screw_link: mass 1.0 -> 1
Joints:
- added joint l_force_torque_adapter_joint: type fixed, parent l_wrist_roll_link, child l_force_torque_adapter_link, origin xyz=0.0356 0 0 rpy=0 -1.570796326795 0
- added joint l_force_torque_joint: type fixed, parent l_force_torque_adapter_link, child l_force_torque_link, origin xyz=0 0 0 rpy=0 0 1.221730476396
- joint base_laser_joint: origin xyz=0.275 0.0 0.252 rpy=0 0 0 -> xyz=0.275 0 0.252 rpy=0 0 0
- joint double_stereo_frame_joint: origin xyz=0.0 0.0 0.0 rpy=0 0 0 -> xyz=0 0 0 rpy=0 0 0
- joint head_mount_kinect_ir_optical_frame_joint: origin xyz=0.0            0.01         0.0 rpy=-1.57079632679 0.0 -1.57079632679 -> xyz=0 0.01 0 rpy=-1.57079632679 0 -1.57079632679
- joint head_mount_kinect_rgb_joint: origin xyz=0 -0.03 0 rpy=0 0 0 -> xyz=-0.016464580011 -0.024840302033 -0.015501555887 rpy=-0.009197234917 -0.03162989289 -0.000024986557
- joint head_mount_kinect_rgb_optical_frame_joint: origin xyz=0.0            0.0         0.0 rpy=-1.57079632679 0.0 -1.57079632679 -> xyz=0 0 0 rpy=-1.57079632679 0 -1.57079632679
- joint head_mount_prosilica_optical_frame_joint: origin xyz=0.0            0.0         0.0 rpy=-1.57079632679 0.0 -1.57079632679 -> xyz=0 0 0 rpy=-1.57079632679 0 -1.57079632679
- joint head_pan_joint: origin xyz=-0.01707 0.0 0.38145 rpy=0.0 0.0 0.0 -> xyz=-0.01707 0 0.38145 rpy=0 0 0
- joint high_def_frame_joint: origin xyz=0.046457 -0.110 0.054600 rpy=0 0 0 -> xyz=0.037305871189 -0.109084466748 0.051107786118 rpy=-0.013344088743 -0.002157650878 0.00598407071
- joint high_def_optical_frame_joint: origin xyz=0.0            0.0         0.0 rpy=-1.57079632679 0.0 -1.57079632679 -> xyz=0 0 0 rpy=-1.57079632679 0 -1.57079632679
- joint l_elbow_flex_joint: limit lower=-2.3213 upper=0.00 effort=30 velocity=3.3 -> lower=-2.3213 upper=0 effort=30 velocity=3.3
- joint l_forearm_cam_frame_joint: origin xyz=.135 0 .044 rpy=-1.57079632679 -0.562868683768 0 -> xyz=0.143534195191 0.005377510982 0.038210342235 rpy=-1.538533018262 -0.563330072035 -0.015596777949
- joint l_forearm_cam_optical_frame_joint: origin xyz=0 0 0 rpy=-1.57079632679 0.0 -1.57079632679 -> xyz=0 0 0 rpy=-1.57079632679 0 -1.57079632679
- joint l_gripper_joint: limit lower=0.0 upper=0.09 effort=1000.0 velocity=0.2 -> lower=0 upper=0.09 effort=1000 velocity=0.2; origin (none) -> xyz=0 0 0 rpy=0 0 0
- joint l_gripper_l_finger_joint: limit lower=0.0 upper=0.548 effort=1000.0 velocity=0.5 -> lower=0 upper=0.548 effort=1000 velocity=0.5
- joint l_gripper_l_finger_tip_joint: limit lower=0.0 upper=0.548 effort=1000.0 velocity=0.5 -> lower=0 upper=0.548 effort=1000 velocity=0.5; mimic joint=l_gripper_l_finger_joint multiplier=1 offset=0 -> (none)
- joint l_gripper_led_joint: origin xyz=0.0513 0.0 .0244 -> xyz=0.0513 0 0.0244 rpy=0 0 0
- joint l_gripper_motor_screw_joint: origin xyz=0.0 0 0 rpy=0 0 0 -> xyz=0 0 0 rpy=0 0 0
- joint l_gripper_motor_slider_joint: limit lower=-0.1 upper=0.1 effort=1000.0 velocity=0.2 -> lower=-0.1 upper=0.1 effort=1000 velocity=0.2
- joint l_gripper_palm_joint: origin xyz=0 0 0 rpy=0 0 0 -> xyz=0 0 0 rpy=0 1.570796326795 -1.221730476396; parent l_wrist_roll_link -> l_force_torque_link
- joint l_gripper_r_finger_joint: limit lower=0.0 upper=0.548 effort=1000.0 velocity=0.5 -> lower=0 upper=0.548 effort=1000 velocity=0.5; mimic joint=l_gripper_l_finger_joint multiplier=1 offset=0 -> (none)
- joint l_gripper_r_finger_tip_joint: limit lower=0.0 upper=0.548 effort=1000.0 velocity=0.5 -> lower=0 upper=0.548 effort=1000 velocity=0.5; mimic joint=l_gripper_l_finger_joint multiplier=1 offset=0 -> (none)
- joint l_shoulder_pan_joint: origin xyz=0.0 0.188 0.0 rpy=0 0 0 -> xyz=0 0.188 0 rpy=0 0 0
- joint l_torso_lift_side_plate_joint: origin xyz=0.0535 0.209285 0.176625 -> xyz=0.0535 0.209285 0.176625 rpy=0 0 0
- joint l_wrist_flex_joint: limit lower=-2.18 upper=0.0 effort=10 velocity=3.078 -> lower=-2.18 upper=0 effort=10 velocity=3.078
- joint laser_tilt_joint: origin xyz=0 0 0.03 rpy=0 0 0 -> xyz=0 0 0.028389479248 rpy=0 0 -0.007935244203
- joint laser_tilt_mount_joint: limit lower=-0.7854 upper=1.48353 effort=0.65 velocity=10.0 -> lower=-0.7854 upper=1.48353 effort=0.65 velocity=10
- joint narrow_stereo_frame_joint: origin xyz=0.045 0.06 0.0501 rpy=0.0   0.0   0.0 -> xyz=0.036004211982 0.059339423616 0.046128460576 rpy=-0.006360148572 -0.007022640169 0.00538386839
- joint narrow_stereo_l_stereo_camera_optical_frame_joint: origin xyz=0 0 0 rpy=-1.57079632679 0.0 -1.57079632679 -> xyz=0 0 0 rpy=-1.57079632679 0 -1.57079632679
- joint narrow_stereo_optical_frame_joint: origin xyz=0 0 0 rpy=-1.57079632679 0.0 -1.57079632679 -> xyz=0 0 0 rpy=-1.57079632679 0 -1.57079632679
- joint narrow_stereo_r_stereo_camera_frame_joint: origin xyz=0.0 -0.09 0.0 rpy=0.0 0.0 0.0 -> xyz=0 -0.09 0 rpy=0 0 0
- joint narrow_stereo_r_stereo_camera_optical_frame_joint: origin xyz=0 0 0 rpy=-1.57079632679 0.0 -1.57079632679 -> xyz=0 0 0 rpy=-1.57079632679 0 -1.57079632679
- joint projector_wg6802418_frame_joint: origin xyz=0 0.110 0.0546 rpy=0 0 0 -> xyz=0 0.11 0.0546 rpy=0 0 0
- joint r_elbow_flex_joint: limit lower=-2.3213 upper=0.00 effort=30 velocity=3.3 -> lower=-2.3213 upper=0 effort=30 velocity=3.3
- joint r_forearm_cam_frame_joint: origin xyz=.135 0 .044 rpy=1.57079632679 -0.562868683768 0 -> xyz=0.138338823418 -0.00626146937 0.044938792621 rpy=1.549884508472 -0.52315633191 0.0073610857
- joint r_forearm_cam_optical_frame_joint: origin xyz=0 0 0 rpy=-1.57079632679 0.0 -1.57079632679 -> xyz=0 0 0 rpy=-1.57079632679 0 -1.57079632679
- joint r_gripper_joint: limit lower=0.0 upper=0.09 effort=1000.0 velocity=0.2 -> lower=0 upper=0.09 effort=1000 velocity=0.2; origin (none) -> xyz=0 0 0 rpy=0 0 0
- joint r_gripper_l_finger_joint: limit lower=0.0 upper=0.548 effort=1000.0 velocity=0.5 -> lower=0 upper=0.548 effort=1000 velocity=0.5
- joint r_gripper_l_finger_tip_joint: limit lower=0.0 upper=0.548 effort=1000.0 velocity=0.5 -> lower=0 upper=0.548 effort=1000 velocity=0.5; mimic joint=r_gripper_l_finger_joint multiplier=1 offset=0 -> (none)
- joint r_gripper_led_joint: origin xyz=0.0513 0.0 .0244 -> xyz=0.0513 0 0.0244 rpy=0 0 0
- joint r_gripper_motor_screw_joint: origin xyz=0.0 0 0 rpy=0 0 0 -> xyz=0 0 0 rpy=0 0 0
- joint r_gripper_motor_slider_joint: limit lower=-0.1 upper=0.1 effort=1000.0 velocity=0.2 -> lower=-0.1 upper=0.1 effort=1000 velocity=0.2
- joint r_gripper_r_finger_joint: limit lower=0.0 upper=0.548 effort=1000.0 velocity=0.5 -> lower=0 upper=0.548 effort=1000 velocity=0.5; mimic joint=r_gripper_l_finger_joint multiplier=1 offset=0 -> (none)
- joint r_gripper_r_finger_tip_joint: limit lower=0.0 upper=0.548 effort=1000.0 velocity=0.5 -> lower=0 upper=0.548 effort=1000 velocity=0.5; mimic joint=r_gripper_l_finger_joint multiplier=1 offset=0 -> (none)
- joint r_shoulder_pan_joint: origin xyz=0.0 -0.188 0.0 rpy=0 0 0 -> xyz=0 -0.188 0 rpy=0 0 0
- joint r_torso_lift_side_plate_joint: origin xyz=0.0535  -0.209285 0.176625 -> xyz=0.0535 -0.209285 0.176625 rpy=0 0 0
- joint r_wrist_flex_joint: limit lower=-2.18 upper=0.0 effort=10 velocity=3.078 -> lower=-2.18 upper=0 effort=10 velocity=3.078
- joint sensor_mount_frame_joint: origin xyz=0.0 0.0 0.0 rpy=0 0 0 -> xyz=0 0 0 rpy=0 0 0
- joint torso_lift_joint: limit lower=0.0 upper=0.33 effort=10000 velocity=0.013 -> lower=0 upper=0.33 effort=10000 velocity=0.013
- joint torso_lift_motor_screw_joint: origin xyz=-0.15 0.0 0.7 -> xyz=-0.15 0 0.7 rpy=0 0 0
- joint wide_stereo_frame_joint: origin xyz=0.045 0.03 0.0501 rpy=0.0   0.0   0.0 -> xyz=0.039047869538 0.028900431683 0.045740529525 rpy=-0.006821150857 -0.011235489405 0.027024041802
- joint wide_stereo_l_stereo_camera_optical_frame_joint: origin xyz=0 0 0 rpy=-1.57079632679 0.0 -1.57079632679 -> xyz=0 0 0 rpy=-1.57079632679 0 -1.57079632679
- joint wide_stereo_optical_frame_joint: origin xyz=0 0 0 rpy=-1.57079632679 0.0 -1.57079632679 -> xyz=0 0 0 rpy=-1.57079632679 0 -1.57079632679
- joint wide_stereo_r_stereo_camera_frame_joint: origin xyz=0.0 -0.09 0.0 rpy=0.0 0.0 0.0 -> xyz=0 -0.09 0 rpy=0 0 0
- joint wide_stereo_r_stereo_camera_optical_frame_joint: origin xyz=0 0 0 rpy=-1.57079632679 0.0 -1.57079632679 -> xyz=0 0 0 rpy=-1.57079632679 0 -1.57079632679
